Commit message: URDF completa, recordar hacer cambios

File: servo_hardware/description/ros2_control/servo.ros2_control.xacro (robot description, xacro)
@@ -1,5 +1,5 @@
 <?xml version="1.0"?>
 <robot xmlns:xacro="http://www.ros.org/wiki/xacro">
-  <xacro:macro name="servo_ros2_control" params="name prefix">
+  <xacro:macro name="servo_ros2_control" params="name">
     <ros2_control name="${name}" type="system">
       <hardware>
@@ -16,6 +16,6 @@
         <param name="pid_o">50</param>
       </hardware>
-      <joint name="${prefix}servo_joint">
-        <command_interface name="position"/>
+      <joint name="servo_joint">
+        <command_interface name="velocity"/>
         <state_interface name="position"/>
         <state_interface name="velocity"/>

Commit message: ros2-control actualizado

File: servo_hardware/description/ros2_control/servo.ros2_control.xacro (robot description, xacro)
@@ -5,5 +5,8 @@
       <hardware>
         <plugin>servo_hardware/ServoArduinoHardware</plugin>
-        <param name="joint1_name">servo_joint</param>
+        <param name="joint1_name">hombro</param>
+        <param name="joint2_name">codo</param>
+        <param name="joint3_name">muneca</param>
+        <param name="joint4_name">articulacion</param>
         <param name="loop_rate">30</param>
         <param name="device">/home/jammy/servo</param>
@@ -16,5 +19,20 @@
         <param name="pid_o">50</param>
       </hardware>
-      <joint name="servo_joint">
+      <joint name="hombro">
+        <command_interface name="velocity"/>
+        <state_interface name="position"/>
+        <state_interface name="velocity"/>
+      </joint>
+      <joint name="codo">
+        <command_interface name="velocity"/>
+        <state_interface name="position"/>
+        <state_interface name="velocity"/>
+      </joint>
+      <joint name="muneca">
+        <command_interface name="velocity"/>
+        <state_interface name="position"/>
+        <state_interface name="velocity"/>
+      </joint>
+      <joint name="articulacion">
         <command_interface name="velocity"/>
         <state_interface name="position"/>

File: servo_hardware/description/urdf/epson_scara.urdf.xacro (robot description, xacro)
@@ -4,5 +4,5 @@
      For more information, please see http://wiki.ros.org/sw_urdf_exporter -->
 <robot
-  name="epson">
+  name="servo_ros2">
   <link
     name="world"/>
@@ -29,5 +29,5 @@
       <geometry>
         <mesh
-          filename="package://epson/meshes/base.STL" />
+          filename="package://servo_ros2/meshes/base.STL" />
       </geometry>
       <material
@@ -43,5 +43,5 @@
       <geometry>
         <mesh
-          filename="package://epson/meshes/base.STL" />
+          filename="package://servo_ros2/meshes/base.STL" />
       </geometry>
     </collision>
@@ -80,5 +80,5 @@
       <geometry>
         <mesh
-          filename="package://epson/meshes/antebrazo.STL" />
+          filename="package://servo_ros2/meshes/antebrazo.STL" />
       </geometry>
       <material
@@ -94,5 +94,5 @@
       <geometry>
         <mesh
-          filename="package://epson/meshes/antebrazo.STL" />
+          filename="package://servo_ros2/meshes/antebrazo.STL" />
       </geometry>
     </collision>
@@ -133,5 +133,5 @@
       <geometry>
         <mesh
-          filename="package://epson/meshes/brazo.STL" />
+          filename="package://servo_ros2/meshes/brazo.STL" />
       </geometry>
       <material
@@ -147,5 +147,5 @@
       <geometry>
         <mesh
-          filename="package://epson/meshes/brazo.STL" />
+          filename="package://servo_ros2/meshes/brazo.STL" />
       </geometry>
     </collision>
@@ -186,5 +186,5 @@
       <geometry>
         <mesh
-          filename="package://epson/meshes/mano.STL" />
+          filename="package://servo_ros2/meshes/mano.STL" />
       </geometry>
       <material
@@ -200,5 +200,5 @@
       <geometry>
         <mesh
-          filename="package://epson/meshes/mano.STL" />
+          filename="package://servo_ros2/meshes/mano.STL" />
       </geometry>
     </collision>
@@ -244,5 +244,5 @@
       <geometry>
         <mesh
-          filename="package://epson/meshes/dedo.STL" />
+          filename="package://servo_ros2/meshes/dedo.STL" />
       </geometry>
       <material
@@ -258,5 +258,5 @@
       <geometry>
         <mesh
-          filename="package://epson/meshes/dedo.STL" />
+          filename="package://servo_ros2/meshes/dedo.STL" />
       </geometry>
     </collision>
