Commit message: no funciona aun.. aun

File: servo_hardware/description/gazebo/servo.gazebo.xacro (robot description, xacro)
@@ -2,8 +2,17 @@
 <robot>
     <!-- Gazebo Colors -->
-    <gazebo reference="motor">
+    <gazebo reference="base_link">
+        <material>Gazebo/White</material>
+    </gazebo>
+    <gazebo reference="antebrazo">
         <material>Gazebo/Blue</material>
     </gazebo>
-    <gazebo reference="arm">
+    <gazebo reference="brazo">
+        <material>Gazebo/Red</material>
+    </gazebo>
+        <gazebo reference="mano">
+        <material>Gazebo/Blue</material>
+    </gazebo>
+    <gazebo reference="dedo">
         <material>Gazebo/White</material>
     </gazebo>
@@ -13,5 +22,38 @@
             <plugin>gazebo_ros2_control/GazeboSystem</plugin>
         </hardware>
-        <joint name="servo_joint">
+        <joint name="hombro">
+            <command_interface name="position">
+                <param name="min">-1.58</param>
+                <param name="max">1.58</param>
+            </command_interface>
+            <state_interface name="position">
+                <param name="initial_value">0</param>
+            </state_interface>
+            <state_interface name="velocity"/>
+            <state_interface name="effort"/>
+        </joint>
+        <joint name="codo">
+            <command_interface name="position">
+                <param name="min">-1.58</param>
+                <param name="max">1.58</param>
+            </command_interface>
+            <state_interface name="position">
+                <param name="initial_value">0</param>
+            </state_interface>
+            <state_interface name="velocity"/>
+            <state_interface name="effort"/>
+        </joint>
+        <joint name="muneca">
+            <command_interface name="position">
+                <param name="min">-1.58</param>
+                <param name="max">1.58</param>
+            </command_interface>
+            <state_interface name="position">
+                <param name="initial_value">0</param>
+            </state_interface>
+            <state_interface name="velocity"/>
+            <state_interface name="effort"/>
+        </joint>
+        <joint name="articulacion">
             <command_interface name="position">
                 <param name="min">-1.58</param>

File: servo_hardware/description/urdf/servo.simulated.xacro (robot description, xacro)
@@ -1,5 +1,5 @@
 <?xml version="1.0"?>
 <robot xmlns:xacro="http://www.ros.org/wiki/xacro" name="servo">
-    <xacro:include filename="$(find servo_hardware)/urdf/servo.description.xacro" />
+    <xacro:include filename="$(find servo_hardware)/urdf/epson_scara.description.xacro" />
     <xacro:include filename="$(find servo_hardware)/gazebo/servo.gazebo.xacro" />
 </robot>

File: servo_hardware/description/urdf/servo.urdf.xacro (robot description, xacro)
@@ -1,5 +1,5 @@
 <?xml version="1.0"?>
 <robot xmlns:xacro="http://www.ros.org/wiki/xacro" name="servo">
-    <xacro:include filename="$(find servo_hardware)/urdf/epson_scara.urdf.xacro" />
+    <xacro:include filename="$(find servo_hardware)/urdf/epson_scara.description.xacro" />
     <xacro:include filename="$(find servo_hardware)/ros2_control/servo.ros2_control.xacro" />
     <xacro:servo_ros2_control name="servo" prefix="" />

File: servo_hardware_moveit_config/config/servo.ros2_control.xacro (robot description, xacro)
@@ -1,9 +1,12 @@
 <?xml version="1.0"?>
 <robot xmlns:xacro="http://www.ros.org/wiki/xacro">
-  <xacro:macro name="servo_ros2_control" params="name prefix plugin">
+  <xacro:macro name="servo_ros2_control" params="name plugin">
     <ros2_control name="${name}" type="system">
       <hardware>
         <plugin>${plugin}</plugin>
-        <param name="joint1_name">servo_joint</param>
+        <param name="joint1_name">hombro</param>
+        <param name="joint2_name">codo</param>
+        <param name="joint3_name">muneca</param>
+        <param name="joint4_name">articulacion</param>
         <param name="loop_rate">30</param>
         <param name="device">/tmp/servo</param>
@@ -16,6 +19,21 @@
         <param name="pid_o">50</param>
       </hardware>
-      <joint name="${prefix}servo_joint">
-        <command_interface name="position"/>
+      <joint name="hombro">
+        <command_interface name="velocity"/>
+        <state_interface name="position"/>
+        <state_interface name="velocity"/>
+      </joint>
+      <joint name="codo">
+        <command_interface name="velocity"/>
+        <state_interface name="position"/>
+        <state_interface name="velocity"/>
+      </joint>
+      <joint name="muneca">
+        <command_interface name="velocity"/>
+        <state_interface name="position"/>
+        <state_interface name="velocity"/>
+      </joint>
+      <joint name="articulacion">
+        <command_interface name="velocity"/>
         <state_interface name="position"/>
         <state_interface name="velocity"/>

File: servo_hardware_moveit_config/config/servo.urdf.xacro (robot description, xacro)
@@ -2,5 +2,5 @@
 <robot xmlns:xacro="http://www.ros.org/wiki/xacro" name="servo">
     <!-- Import panda urdf file -->
-    <xacro:include filename="$(find servo_hardware)/urdf/servo.description.xacro" />
+    <xacro:include filename="$(find servo_hardware)/urdf/epson_scara.description.xacro" />
     <!-- Import servo ros2_control description -->
     <xacro:include filename="servo.ros2_control.xacro" />
@@ -8,5 +8,4 @@
         name="servo"
         plugin="servo_hardware/ServoArduinoHardware"
-        prefix=""
     />
 </robot>

File: servo_hardware_moveit_config/config/servo_gazebo.urdf.xacro (robot description, xacro)
@@ -2,5 +2,5 @@
 <robot xmlns:xacro="http://www.ros.org/wiki/xacro" name="servo">
     <!-- Import panda urdf file -->
-    <xacro:include filename="$(find servo_hardware)/urdf/servo.description.xacro" />
+    <xacro:include filename="$(find servo_hardware)/urdf/epson_scara.description.xacro" />
     <!-- Import servo ros2_control description -->
     <xacro:include filename="servo.ros2_control.xacro" />
@@ -11,8 +11,18 @@
     />
     <!-- Gazebo Colors & Plugins -->
-    <gazebo reference="motor">
+    </gazebo>
+        <gazebo reference="base_link">
+        <material>Gazebo/White</material>
+    </gazebo>
+    <gazebo reference="antebrazo">
         <material>Gazebo/Blue</material>
     </gazebo>
-    <gazebo reference="arm">
+    <gazebo reference="brazo">
+        <material>Gazebo/Red</material>
+    </gazebo>
+        <gazebo reference="mano">
+        <material>Gazebo/Blue</material>
+    </gazebo>
+    <gazebo reference="dedo">
         <material>Gazebo/White</material>
     </gazebo>

File: servo_hardware_moveit_config/config/servo_mock.urdf.xacro (robot description, xacro)
@@ -2,5 +2,5 @@
 <robot xmlns:xacro="http://www.ros.org/wiki/xacro" name="servo">
     <!-- Import panda urdf file -->
-    <xacro:include filename="$(find servo_hardware)/urdf/servo.description.xacro" />
+    <xacro:include filename="$(find servo_hardware)/urdf/epson_scara.description.xacro" />
     <!-- Import servo ros2_control description -->
     <xacro:include filename="servo.ros2_control.xacro" />
@@ -8,5 +8,4 @@
         name="servo"
         plugin="mock_components/GenericSystem"
-        prefix=""
     />
 </robot>
