Commit message: ya se muestra completa faltapaquete de controllers

File: servo_hardware/description/urdf/epson_scara.description.xacro (robot description, xacro)
@@ -23,5 +23,5 @@
             <origin xyz="0 0 0" rpy="0 0 0" />
             <geometry>
-                <mesh filename="package://servo_harware/meshes/base.STL" />
+                <mesh filename="package://servo_hardware/meshes/base.STL" />
             </geometry>
         </collision>
@@ -41,5 +41,5 @@
             <origin xyz="0 0 0" rpy="0 0 0" />
             <geometry>
-                <mesh filename="package://servo_harware/meshes/antebrazo.STL" />
+                <mesh filename="package://servo_hardware/meshes/antebrazo.STL" />
             </geometry>
             <material name="">
@@ -50,5 +50,5 @@
             <origin xyz="0 0 0" rpy="0 0 0" />
             <geometry>
-                <mesh filename="package://servo_harware/meshes/antebrazo.STL" />
+                <mesh filename="package://servo_hardware/meshes/antebrazo.STL" />
             </geometry>
         </collision>
@@ -69,5 +69,5 @@
             <origin xyz="0 0 0" rpy="0 0 0" />
             <geometry>
-                <mesh filename="package://servo_harware/meshes/brazo.STL" />
+                <mesh filename="package://servo_hardware/meshes/brazo.STL" />
             </geometry>
             <material name="">
@@ -78,5 +78,5 @@
             <origin xyz="0 0 0" rpy="0 0 0" />
             <geometry>
-                <mesh filename="package://servo_harware/meshes/brazo.STL" />
+                <mesh filename="package://servo_hardware/meshes/brazo.STL" />
             </geometry>
         </collision>
@@ -97,5 +97,5 @@
             <origin xyz="0 0 0" rpy="0 0 0" />
             <geometry>
-                <mesh filename="package://servo_harware/meshes/mano.STL" />
+                <mesh filename="package://servo_hardware/meshes/mano.STL" />
             </geometry>
             <material name="">
@@ -106,5 +106,5 @@
             <origin xyz="0 0 0" rpy="0 0 0" />
             <geometry>
-                <mesh filename="package://servo_harware/meshes/mano.STL" />
+                <mesh filename="package://servo_hardware/meshes/mano.STL" />
             </geometry>
         </collision>
@@ -126,5 +126,5 @@
             <origin xyz="0 0 0" rpy="0 0 0" />
             <geometry>
-                <mesh filename="package://servo_harware/meshes/dedo.STL" />
+                <mesh filename="package://servo_hardware/meshes/dedo.STL" />
             </geometry>
             <material name="">
@@ -135,5 +135,5 @@
             <origin xyz="0 0 0" rpy="0 0 0" />
             <geometry>
-                <mesh filename="package://servo_harware/meshes/dedo.STL" />
+                <mesh filename="package://servo_hardware/meshes/dedo.STL" />
             </geometry>
         </collision>

File: servo_hardware_moveit_config/config/servo.urdf.xacro (robot description, xacro)
@@ -1,4 +1,4 @@
 <?xml version="1.0"?>
-<robot xmlns:xacro="http://www.ros.org/wiki/xacro" name="servo">
+<robot xmlns:xacro="http://www.ros.org/wiki/xacro" name="servo_ros2">
     <!-- Import panda urdf file -->
     <xacro:include filename="$(find servo_hardware)/urdf/epson_scara.description.xacro" />

File: servo_hardware_moveit_config/config/servo_gazebo.urdf.xacro (robot description, xacro)
@@ -1,4 +1,4 @@
 <?xml version="1.0"?>
-<robot xmlns:xacro="http://www.ros.org/wiki/xacro" name="servo">
+<robot xmlns:xacro="http://www.ros.org/wiki/xacro" name="servo_ros2">
     <!-- Import panda urdf file -->
     <xacro:include filename="$(find servo_hardware)/urdf/epson_scara.description.xacro" />

File: servo_hardware_moveit_config/config/servo_mock.urdf.xacro (robot description, xacro)
@@ -1,4 +1,4 @@
 <?xml version="1.0"?>
-<robot xmlns:xacro="http://www.ros.org/wiki/xacro" name="servo">
+<robot xmlns:xacro="http://www.ros.org/wiki/xacro" name="servo_ros2">
     <!-- Import panda urdf file -->
     <xacro:include filename="$(find servo_hardware)/urdf/epson_scara.description.xacro" />
