Commit message: Depurado y funcionando

File: scara_hardware/config/ros2_control.xacro (robot description, xacro)
@@ -1,5 +1,5 @@
 <?xml version="1.0"?>
 <robot xmlns:xacro="http://www.ros.org/wiki/xacro">
-  <xacro:macro name="servo_ros2_control" params="name plugin">
+  <xacro:macro name="hardware_component" params="name plugin">
     <ros2_control name="${name}" type="system">
       <hardware>
@@ -31,5 +31,5 @@
         <!-- Serial Communication -->
         <param name="loop_rate">30</param>
-        <param name="device">/tmp/scara</param>
+        <param name="device">/home/jammy/servo</param>
         <param name="baud_rate">115200</param>
         <param name="timeout_ms">1000</param>
@@ -37,21 +37,37 @@
       <joint name="hombro">
         <command_interface name="position"/>
-        <state_interface name="position"/>
-        <state_interface name="velocity"/>
+        <state_interface name="position">
+          <param name="initial_value">0.0</param>
+        </state_interface>
+        <state_interface name="velocity">
+          <param name="initial_value">0.0</param>
+        </state_interface>
       </joint>
       <joint name="codo">
         <command_interface name="position"/>
-        <state_interface name="position"/>
-        <state_interface name="velocity"/>
+        <state_interface name="position">
+          <param name="initial_value">0.0</param>
+        </state_interface>
+        <state_interface name="velocity">
+          <param name="initial_value">0.0</param>
+        </state_interface>
       </joint>
       <joint name="muneca">
         <command_interface name="position"/>
-        <state_interface name="position"/>
-        <state_interface name="velocity"/>
+        <state_interface name="position">
+          <param name="initial_value">0.0</param>
+        </state_interface>
+        <state_interface name="velocity">
+          <param name="initial_value">0.0</param>
+        </state_interface>
       </joint>
       <joint name="articulacion">
         <command_interface name="position"/>
-        <state_interface name="position"/>
-        <state_interface name="velocity"/>
+        <state_interface name="position">
+          <param name="initial_value">0.0</param>
+        </state_interface>
+        <state_interface name="velocity">
+          <param name="initial_value">0.0</param>
+        </state_interface>
       </joint>
     </ros2_control>

File: servo_hardware_moveit_config/config/servo.urdf.xacro (robot description, xacro)
@@ -4,7 +4,7 @@
     <xacro:include filename="$(find servo_hardware)/urdf/epson_scara.description.xacro" />
     <!-- Import servo ros2_control description -->
-    <xacro:include filename="servo.ros2_control.xacro" />
-    <xacro:servo_ros2_control
-        name="servo"
+    <xacro:include filename="$(find scara_hardware)/config/ros2_control.xacro" />
+    <xacro:hardware_component
+        name="hardware_component"
         plugin="scara_hardware/ScaraHardwareComponent"
     />

File: servo_hardware_moveit_config/config/servo_gazebo.urdf.xacro (robot description, xacro)
@@ -1,32 +1,5 @@
 <?xml version="1.0"?>
 <robot xmlns:xacro="http://www.ros.org/wiki/xacro" name="servo_ros2">
-    <!-- Import panda urdf file -->
-    <xacro:include filename="$(find servo_hardware)/urdf/epson_scara.description.xacro" />
-    <!-- Import servo ros2_control description -->
-    <xacro:include filename="servo.ros2_control.xacro" />
-    <xacro:servo_ros2_control
-        name="servo"
-        plugin="gazebo_ros2_control/GazeboSystem"
-    />
-    <!-- Gazebo Colors & Plugins -->
-    <gazebo reference="base_link">
-        <material>Gazebo/White</material>
-    </gazebo>
-    <gazebo reference="antebrazo">
-        <material>Gazebo/Blue</material>
-    </gazebo>
-    <gazebo reference="brazo">
-        <material>Gazebo/Red</material>
-    </gazebo>
-        <gazebo reference="mano">
-        <material>Gazebo/Blue</material>
-    </gazebo>
-    <gazebo reference="dedo">
-        <material>Gazebo/White</material>
-    </gazebo>
-    <gazebo>
-        <plugin filename="libgazebo_ros2_control.so" name="gazebo_ros2_control">
-            <parameters>$(find servo_hardware_moveit_config)/config/ros2_controllers.yaml</parameters>
-        </plugin>
-    </gazebo>
+    <!-- Import scara urdf file -->
+    <xacro:include filename="$(find servo_hardware)/urdf/servo.gazebo.xacro" />
 </robot>

File: servo_hardware_moveit_config/config/servo_mock.urdf.xacro (robot description, xacro)
@@ -4,8 +4,8 @@
     <xacro:include filename="$(find servo_hardware)/urdf/epson_scara.description.xacro" />
     <!-- Import servo ros2_control description -->
-    <xacro:include filename="servo.ros2_control.xacro" />
-    <xacro:servo_ros2_control
-        name="servo"
-        plugin="mock_components/GenericSystem"
+    <xacro:include filename="$(find scara_hardware)/config/ros2_control.xacro" />
+    <xacro:hardware_component
+        name="hardware_component"
+        plugin="scara_hardware/ScaraHardwareComponent"
     />
 </robot>
